File: Hardware/Qwiic_Spectral_Sensor_AS7341.sch (EAGLE design)
At the start: 36 parts, among them J1 QWIIC_RIGHT_ANGLE, J3 QWIIC_RIGHT_ANGLE, Q1 20V/4.2A/52mΩ/1.4W, Q2 20V/4.2A/52mΩ/1.4W, Q3 20V/4.2A/52mΩ/1.4W, U1 AS7341OLGA, U2 PCA9536, U3 AP2127K-1.8V

Commit message: added as7341 decoupling cap
Parts:
- added C5: 0.1uF, SparkFun-Capacitors:0.1UF-0603-25V-(+80/-20%)
Connections:
- net 1.8V: now also C5.1
- net GND: now also C5.2
Changed lines of the file:
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@@
 <part name="GND3" library="SparkFun-PowerSymbols" deviceset="GND" device=""/>
 <part name="SUPPLY2" library="SparkFun-PowerSymbols" deviceset="3.3V" device=""/>
+<part name="C5" library="SparkFun-Capacitors" deviceset="0.1UF" device="-0603-25V-(+80/-20%)" value="0.1uF"/>
+<part name="GND12" library="SparkFun-PowerSymbols" deviceset="GND" device=""/>
+<part name="SUPPLY17" library="SparkFun-PowerSymbols" deviceset="1.8V" device=""/>
 </parts>
 <sheets>
@@
 <attribute name="VALUE" x="109.22" y="40.894" size="1.778" layer="96" align="bottom-center"/>
 </instance>
+<instance part="C5" gate="G$1" x="12.7" y="157.48" smashed="yes">
+<attribute name="NAME" x="14.224" y="160.401" size="1.778" layer="95" font="vector"/>
+<attribute name="VALUE" x="14.224" y="155.321" size="1.778" layer="96" font="vector"/>
+</instance>
+<instance part="GND12" gate="1" x="12.7" y="149.86" smashed="yes">
+<attribute name="VALUE" x="12.7" y="149.606" size="1.778" layer="96" align="top-center"/>
+</instance>
+<instance part="SUPPLY17" gate="G$1" x="12.7" y="165.1" smashed="yes">
+<attribute name="VALUE" x="12.7" y="167.894" size="1.778" layer="96" align="bottom-center"/>
+</instance>
 </instances>
 <busses>
@@
 <pinref part="GND3" gate="1" pin="GND"/>
 </segment>
+<segment>
+<pinref part="C5" gate="G$1" pin="2"/>
+<pinref part="GND12" gate="1" pin="GND"/>
+<wire x1="12.7" y1="152.4" x2="12.7" y2="154.94" width="0.1524" layer="91"/>
+</segment>
 </net>
 <net name="N$4" class="0">
@@
 <pinref part="SUPPLY16" gate="G$1" pin="1.8V"/>
 </segment>
-</net>
+<segment>
+<pinref part="C5" gate="G$1" pin="1"/>
+<pinref part="SUPPLY17" gate="G$1" pin="1.8V"/>
+<wire x1="12.7" y1="165.1" x2="12.7" y2="162.56" width="0.1524" layer="91"/>
+</segment>
+</net>

Commit message: Board design
Parts:
- J2: device SparkFun-Connectors:CONN_05NO_SILK -> SparkFun-Connectors:CONN_06NO_SILK_FEMALE_PTH
Connections:
- net INT renamed !INT!
- removed net N$6: U3.EN, U3.IN
- net 3.3V: now also Q1.S, Q2.S, U3.EN, U3.IN; no longer Q1.D, Q2.D
- net GPIO3: now also J2.6, U1.GPIO
- net N$8: now also Q1.D; no longer Q1.S
- net N$9: now also Q2.D; no longer Q2.S
Other:
- note added: "LEDs"
- note removed: "LED's"
- moved on the sheet: Q1, Q2, R4, U1

Commit message: Board review notes
Parts:
- added JP5: JUMPER-SMT_2_NC_TRACE_SILK, SparkFun-Jumpers:JUMPER-SMT_2_NC_TRACE_SILK
- added R5: 2.2k, SparkFun-Resistors:2.2KOHM-0603-1/10W-1%
Connections:
- new net N$6: JP2.2, Q3.D
- net !INT!: now also U1.!INT!; no longer U1.INT
- net 1.8V: now also JP5.2; no longer R4.2
- net 3.3V: now also Q3.S; no longer Q3.D
- net GND: now also R5.1
- net GPIO0: now also R5.2
- net GPIO3: no longer U2.GPIO3
- net N$10: now also JP5.1, R4.2; no longer JP2.2, Q3.S
Other:
- note added: "Cut jumpers 3 and 4 to use specialized LED bulbs and solder them to through-hole footprints of D4 and/or D5."
- moved on the sheet: C5, D1, JP2, Q3, R3, R4, U1

Commit message: Add schematic.
Parts:
- added LOGO1: QWIIC_LOGO_6MM, SparkFun-Aesthetics:QWIIC_LOGO_6MM
- added U$31: SPARKX-LOGO3, SparkX:SPARKX-LOGO3
Other:
- note added: "Power LED"
- note removed: "PWR LED"
- moved on the sheet: D1, JP2, Q3, R3, R5
